Commit message: urdf finished

File: src/giraffe_files/urdf/giraffe_robot.urdf.xacro (robot description, xacro)
@@ -3,9 +3,7 @@
     <!-- parameters -->
     <xacro:property name="ceiling_height" value="4.0"/>
-    <xacro:property name="base_radius" value="0.1"/>
-    <xacro:property name="base_length" value="0.1"/>
     <xacro:property name="link_radius" value="0.05"/>
-    <xacro:property name="prismatic_length" value="3.0"/>  <!-- prismatic range -->
-    <xacro:property name="wrist_length" value="0.2"/>
+    <xacro:property name="prismatic_length" value="5.5"/>  <!-- prismatic range -->
+    <xacro:property name="wrist_length" value="1"/>
     <!-- materials -->
     <!-- grey for links, blue for joints -->
@@ -16,6 +14,27 @@
         <color rgba="0.5 0.5 0.5 1"/>
     </material>
+    <material name="White">
+        <color rgba="1 1 1 1"/>
+    </material>
+    <material name="Black">
+        <color rgba="0 0 0 1"/>
+    </material>
+    <link name="world"/>
+    <!-- floor 5x12 -->
+    <link name="floor">
+    <visual>
+        <geometry>
+        <box size="5 12 0.01"/> <!-- thin plane -->
+        </geometry>
+        <origin xyz="2.5 6 0" rpy="0 0 0"/>
+        <material name="Grey"/>
+    </visual>
+    </link>
+    <joint name="world_floor" type="fixed">
+    <parent link="world"/>
+    <child link="floor"/>
+    <origin xyz="0 0 0" rpy="0 0 0"/>
+    </joint>
     <!-- world reference set at the center of the ceiling-->
-    <link name="world"/>
     <joint name="world_base" type="fixed">
         <parent link="world"/>
@@ -36,7 +55,7 @@
         <visual>
             <geometry>
-                <cylinder length="0.1" radius="${link_radius}"/>
+                <sphere radius="${link_radius}"/>
             </geometry>
-            <material name="Blue"/>
+            <material name="White"/>
         </visual>
     </link>
@@ -46,5 +65,5 @@
         <origin xyz="0 0 0" rpy="0 0 0"/>
         <axis xyz="0 0 1"/>
-        <limit lower="-3.14" upper="3.14" effort="10" velocity="1"/>
+        <limit lower="-${pi}" upper="${pi}" effort="10" velocity="1"/>
     </joint>
     <!-- pitch link (y axis) and joint -->
@@ -52,7 +71,8 @@
         <visual>
             <geometry>
-                <cylinder length="0.1" radius="${link_radius}"/>
+                <sphere radius="${link_radius}"/>
             </geometry>
-             <material name="Blue"/>
+            <origin xyz="0 0 0" rpy="0 ${pi/2} 0"/>
+            <material name="White"/>
         </visual>
     </link>
@@ -62,5 +82,5 @@
         <origin xyz="0 0 0" rpy="0 0 0"/>
         <axis xyz="0 1 0"/>
-        <limit lower="-1.57" upper="1.57" effort="10" velocity="1"/>
+        <limit lower="-${1*pi/3}" upper="0" effort="10" velocity="1"/> <!-- 30 degrees is enough, no need to arrive to the ceiling -->
     </joint>
     <!-- prismatic link and joint -->
@@ -71,5 +91,5 @@
                 <cylinder length="${prismatic_length}" radius="${link_radius}"/>
             </geometry>
-            <material name="Blue"/>
+            <material name="White"/>
         </visual>
     </link>
@@ -78,8 +98,8 @@
         <child link="prismatic_link"/>
         <origin xyz="0 0 0" rpy="0 0 0"/>
-        <axis xyz="0 0 -1"/>
+        <axis xyz="0 0 1"/>
         <limit lower="0.0" upper="${prismatic_length}" effort="100" velocity="0.5"/>
     </joint>
-    <!-- wrist link and 2 joints -->
+    <!-- microphone wrist link and 2 joints -->
     <link name="wrist1_link">
         <visual>
@@ -87,5 +107,6 @@
                 <cylinder length="${wrist_length}" radius="${link_radius}"/>
             </geometry>
-            <material name="Grey"/>
+            <origin xyz="0 0 -${wrist_length/2}" rpy="0 0 0"/>
+            <material name="White"/>
         </visual>
     </link>
@@ -93,7 +114,7 @@
         <parent link="prismatic_link"/>
         <child link="wrist1_link"/>
-        <origin xyz="0 0 -${prismatic_length/2}" rpy="0 0 0"/>
+        <origin xyz="0 0 -${prismatic_length}" rpy="0 0 0"/>
         <axis xyz="0 1 0"/>
-        <limit lower="-1.57" upper="1.57" effort="5" velocity="1"/>
+        <limit lower="-${pi/2}" upper="${pi/2}" effort="5" velocity="1"/>
     </joint>
     <joint name="wrist2" type="revolute">
@@ -101,14 +122,28 @@
         <child link="microphone"/>
         <origin xyz="0 0 -${wrist_length}" rpy="0 0 0"/>
-        <axis xyz="1 0 0"/>
-        <limit lower="-1.57" upper="1.57" effort="5" velocity="1"/>
+        <axis xyz="0 1 0"/>
+        <limit lower="-${pi/2}" upper="${pi/2}" effort="5" velocity="1"/>
     </joint>
-    <!-- microphone orientation (end effector) -->
+    <!-- microphone (end effector) -->
      <link name="microphone">
         <visual>
             <geometry>
-                <sphere radius="0.05"/>
+                <sphere radius="0.015"/>
             </geometry>
+            <material name="Black"/>
+        </visual>
+        <visual>
+            <geometry>
+                <cylinder length="0.1" radius="0.02"/>
+            </geometry>
+            <origin xyz="0 0 -0.065" rpy="0 0 0"/>
             <material name="Grey"/>
+        </visual>
+        <visual>
+            <geometry>
+                <sphere radius="0.03"/>
+            </geometry>
+            <origin xyz="0 0 -0.145" rpy="0 0 0"/>
+            <material name="Black"/>
         </visual>
     </link>
