Commit message: urdf changes, direct kinematics, main fixed

File: src/giraffe_files/urdf/giraffe_robot.urdf (robot description, URDF)
Before this commit: robot giraffe_robot, 8 links, 7 joints
Links:
- added link wrist2_link; visual sphere radius=0.015
- link microphone: geometry visual cylinder length=0.1 radius=0.02; visual sphere radius=0.03
Joints:
- added joint mic_frame: type fixed, parent wrist2_link, child microphone, origin xyz=0 0 -0.175 rpy=0 0 0
- joint pitch_joint: limit lower=-1.0471975511965976 upper=0 effort=10 velocity=1 -> lower=-1.5707963267948966 upper=1.5707963267948966 effort=10 velocity=1
- joint prismatic_joint: origin xyz=0 0 0 rpy=0 0 0 -> xyz=0 0 -2.75 rpy=0 0 0
- joint wrist1: origin xyz=0 0 -5.5 rpy=0 0 0 -> xyz=0 0 -2.75 rpy=0 0 0
- joint wrist2: child microphone -> wrist2_link
- joint yaw_joint: origin xyz=0 0 0 rpy=0 0 0 -> xyz=0.0 0.0 -0.07500000000000001 rpy=0 0 0

File: src/giraffe_files/urdf/giraffe_robot.xacro (robot description, xacro)
@@ -3,7 +3,9 @@
     <!-- parameters -->
     <xacro:property name="ceiling_height" value="4.0"/>
+    <xacro:property name="box_heigth" value="0.05"/>
     <xacro:property name="link_radius" value="0.05"/>
     <xacro:property name="prismatic_length" value="5.5"/>  <!-- prismatic range -->
     <xacro:property name="wrist_length" value="1"/>
+    <xacro:property name="wrist2_radius" value="0.015"/>
     <!-- materials -->
     <!-- grey for links, blue for joints -->
@@ -21,5 +23,5 @@
     </material>
     <link name="world"/>
-    <!-- floor 5x12 -->
+   <!--floor 5x12 -->
     <link name="floor">
     <visual>
@@ -27,13 +29,22 @@
         <box size="5 12 0.01"/> <!-- thin plane -->
         </geometry>
-        <origin xyz="2.5 6 0" rpy="0 0 0"/>
+        <origin xyz="2.5 6 -0.005" rpy="0 0 0"/>    <!-- in -z to perfectly center it -->
         <material name="Grey"/>
     </visual>
+    </link >
+    <joint name="world_floor" type="fixed">
+        <parent link="world"/>
+        <child link="floor"/>
+        <origin xyz="0 0 0" rpy="0 0 0"/>
+    </joint>
+    <!-- base link (on the ceiling) -->
+    <link name="base_link">
+        <visual>
+            <geometry>
+                <box size="0.2 0.2 ${box_heigth}"/>
+            </geometry>
+            <material name="Grey"/>
+        </visual>
     </link>
-    <joint name="world_floor" type="fixed">
-    <parent link="world"/>
-    <child link="floor"/>
-    <origin xyz="0 0 0" rpy="0 0 0"/>
-    </joint>
     <!-- world reference set at the center of the ceiling-->
     <joint name="world_base" type="fixed">
@@ -42,13 +53,4 @@
         <origin xyz="2.5 6.0 ${ceiling_height}" rpy="0 0 0"/>
     </joint>
-    <!-- base link (on the ceiling) -->
-    <link name="base_link">
-        <visual>
-            <geometry>
-                <box size="0.2 0.2 0.05"/>
-            </geometry>
-            <material name="Grey"/>
-        </visual>
-    </link>
     <!-- yaw link (z axis) and joint -->
     <link name="yaw_link">
@@ -63,5 +65,5 @@
         <parent link="base_link"/>
         <child link="yaw_link"/>
-        <origin xyz="0 0 0" rpy="0 0 0"/>
+        <origin xyz="0.0 0.0 -${link_radius+box_heigth/2}" rpy="0 0 0"/>
         <axis xyz="0 0 1"/>
         <limit lower="-${pi}" upper="${pi}" effort="10" velocity="1"/>
@@ -82,13 +84,13 @@
         <origin xyz="0 0 0" rpy="0 0 0"/>
         <axis xyz="0 1 0"/>
-        <limit lower="-${1*pi/3}" upper="0" effort="10" velocity="1"/> <!-- 30 degrees is enough, no need to arrive to the ceiling -->
+        <limit lower="-${pi/2}" upper="${pi/2}" effort="10" velocity="1"/> <!-- 30 degrees is enough, no need to arrive to the ceiling -->
     </joint>
     <!-- prismatic link and joint -->
     <link name="prismatic_link">
         <visual>
-            <origin xyz="0 0 -${prismatic_length/2}" rpy="0 0 0"/>
             <geometry>
                 <cylinder length="${prismatic_length}" radius="${link_radius}"/>
             </geometry>
+            <origin xyz="0 0 -${link_radius}" rpy="0 0 0"/>
             <material name="White"/>
         </visual>
@@ -97,9 +99,9 @@
         <parent link="pitch_link"/>
         <child link="prismatic_link"/>
-        <origin xyz="0 0 0" rpy="0 0 0"/>
+        <origin xyz="0 0 -${prismatic_length/2}" rpy="0 0 0"/>
         <axis xyz="0 0 1"/>
         <limit lower="0.0" upper="${prismatic_length}" effort="100" velocity="0.5"/>
     </joint>
-    <!-- microphone wrist link and 2 joints -->
+    <!-- wrist1 link and joint -->
     <link name="wrist1_link">
         <visual>
@@ -114,11 +116,20 @@
         <parent link="prismatic_link"/>
         <child link="wrist1_link"/>
-        <origin xyz="0 0 -${prismatic_length}" rpy="0 0 0"/>
+        <origin xyz="0 0 -${prismatic_length/2}" rpy="0 0 0"/>
         <axis xyz="0 1 0"/>
         <limit lower="-${pi/2}" upper="${pi/2}" effort="5" velocity="1"/>
     </joint>
+    <!-- wrist2 link and joint -->
+    <link name="wrist2_link">
+        <visual>
+            <geometry>
+                <sphere radius="${wrist2_radius}"/>
+            </geometry>
+            <material name="Black"/>
+        </visual>
+    </link>
     <joint name="wrist2" type="revolute">
         <parent link="wrist1_link"/>
-        <child link="microphone"/>
+        <child link="wrist2_link"/>
         <origin xyz="0 0 -${wrist_length}" rpy="0 0 0"/>
         <axis xyz="0 1 0"/>
@@ -129,13 +140,7 @@
         <visual>
             <geometry>
-                <sphere radius="0.015"/>
-            </geometry>
-            <material name="Black"/>
-        </visual>
-        <visual>
-            <geometry>
                 <cylinder length="0.1" radius="0.02"/>
             </geometry>
-            <origin xyz="0 0 -0.065" rpy="0 0 0"/>
+            <origin xyz="0 0 0.11" rpy="0 0 0"/>
             <material name="Grey"/>
         </visual>
@@ -144,7 +149,12 @@
                 <sphere radius="0.03"/>
             </geometry>
-            <origin xyz="0 0 -0.145" rpy="0 0 0"/>
+            <origin xyz="0 0 0.03" rpy="0 0 0"/>
             <material name="Black"/>
         </visual>
     </link>
+    <joint name="mic_frame" type="fixed">
+        <parent link="wrist2_link"/>
+        <child link="microphone"/>
+        <origin xyz="0 0 -0.175" rpy="0 0 0"/>
+    </joint>
 </robot>

Commit message: dynamics code added, inertia added to urdf. Fixes to do

File: src/giraffe_files/urdf/giraffe_robot.urdf (robot description, URDF)
Before this commit: robot giraffe_robot, 9 links, 8 joints
Links:
- link microphone: mass None -> 0.24592387292300896
- link pitch_link: mass None -> 0.7068583470577036
- link prismatic_link: mass None -> 116.6316272645211
- link wrist1_link: mass None -> 21.20575041173111
- link wrist2_link: mass None -> 0.03817035074111598
- link yaw_link: mass None -> 0.7068583470577036

File: src/giraffe_files/urdf/giraffe_robot.xacro (robot description, xacro)
@@ -9,5 +9,4 @@
     <xacro:property name="wrist2_radius" value="0.015"/>
     <!-- materials -->
-    <!-- grey for links, blue for joints -->
     <material name="Blue">
         <color rgba="0 0 0.8 1"/>
@@ -22,4 +21,15 @@
         <color rgba="0 0 0 1"/>
     </material>
+    <!-- params for inertia -->
+    <!-- chosen material for the robot: aluminum. ABS plastic for microphone -->
+    <xacro:property name="density_aluminum" value="2700.0"/>  <!-- density to compute mass (kg/m^3)-->
+    <xacro:property name="density_plastic" value="1030.0"/>  <!-- density to compute mass (kg/m^3)-->
+    <!-- masses of robot elements: density*volume -->
+    <xacro:property name="base_joint_mass" value="${density_aluminum * (4/3)*pi*pow(link_radius, 3)}"/>    <!-- unique sphere volume for joint 1 and 2 -->
+    <xacro:property name="prismatic_mass" value="${density_aluminum * pi*pow(link_radius, 2)*prismatic_length}"/>     <!-- sphere volume -->
+    <xacro:property name="wrist1_joint_mass" value="${density_aluminum* pi*pow(link_radius, 2)*wrist_length}"/>  <!-- cylinder volume -->
+    <xacro:property name="wrist1_mass" value="${density_aluminum* pi*pow(link_radius, 2)*wrist_length}"/>        <!-- cylinder volume -->
+    <xacro:property name="wrist2_joint_mass" value="${density_aluminum* (4/3)*pi*pow(wrist2_radius, 3)}"/>  <!-- sphere volume -->
+    <xacro:property name="mic_mass" value="${density_plastic* ((4/3)*pi*pow(0.03, 3) + pi*pow(0.02, 2)*0.1)}"/>    <!-- cylinder+sphere volume -->
     <link name="world"/>
    <!--floor 5x12 -->
@@ -61,4 +71,14 @@
             <material name="White"/>
         </visual>
+        <inertial>
+            <mass value="${base_joint_mass/2}"/>
+            <origin xyz="0.0 0.0 0.0" rpy="0 0 0"/> <!-- position in the center -->
+            <inertia ixx="${(2.0/5.0) * base_joint_mass * pow(link_radius, 2)}"
+            ixy="0.0"
+            ixz="0.0"
+            iyy="${(2.0/5.0) * base_joint_mass * pow(link_radius, 2)}"
+            iyz="0.0"
+            izz="${(2.0/5.0) * base_joint_mass * pow(link_radius, 2)}"/>   <!-- inertia formula for full spheres -->
+        </inertial>
     </link>
     <joint name="yaw_joint" type="revolute">
@@ -78,4 +98,14 @@
             <material name="White"/>
         </visual>
+        <inertial>
+            <mass value="${base_joint_mass/2}"/>
+            <origin xyz="0.0 0.0 0.0" rpy="0 0 0"/> <!-- position in the center -->
+            <inertia ixx="${(2.0/5.0) * base_joint_mass * pow(link_radius, 2)}"
+            ixy="0.0"
+            ixz="0.0"
+            iyy="${(2.0/5.0) * base_joint_mass * pow(link_radius, 2)}"
+            iyz="0.0"
+            izz="${(2.0/5.0) * base_joint_mass * pow(link_radius, 2)}"/>   <!-- inertia formula for spheres -->
+        </inertial>
     </link>
     <joint name="pitch_joint" type="revolute">
@@ -84,5 +114,5 @@
         <origin xyz="0 0 0" rpy="0 0 0"/>
         <axis xyz="0 1 0"/>
-        <limit lower="-${pi/2}" upper="${pi/2}" effort="10" velocity="1"/> <!-- 30 degrees is enough, no need to arrive to the ceiling -->
+        <limit lower="-${pi/2}" upper="${pi/2}" effort="10" velocity="1"/>
     </joint>
     <!-- prismatic link and joint -->
@@ -95,4 +125,14 @@
             <material name="White"/>
         </visual>
+        <inertial>
+            <mass value="${prismatic_mass}"/>
+            <origin xyz="0.0 0.0 -${prismatic_length/2}" rpy="0 0 0"/> <!-- position in the center -->
+            <inertia ixx="${(1.0/12.0) * prismatic_mass * (3*pow(link_radius,2) + pow(prismatic_length, 2))}"
+            ixy="0.0"
+            ixz="0.0"
+            iyy="${(1.0/12.0) * prismatic_mass * (3*pow(link_radius,2) + pow(prismatic_length, 2))}"
+            iyz="0.0"
+            izz="${(1.0/2.0) * prismatic_mass * pow(link_radius, 2)}"/>   <!-- inertia formula for cylinders (cylinder axis along z) -->
+        </inertial>                                                       <!-- izz=1/2mr^2 , ixx=iyy=1/12m(3r^2+L^2)-->
     </link>
     <joint name="prismatic_joint" type="prismatic">
@@ -112,4 +152,14 @@
             <material name="White"/>
         </visual>
+        <inertial>
+            <mass value="${wrist1_mass}"/>
+            <origin xyz="0.0 0.0 -${wrist_length/2}" rpy="0 0 0"/> <!-- position in the center -->
+            <inertia ixx="${(1.0/12.0) * wrist1_mass * (3*pow(link_radius,2) + pow(wrist_length, 2))}"
+            ixy="0.0"
+            ixz="0.0"
+            iyy="${(1.0/12.0) * wrist1_mass * (3*pow(link_radius,2) + pow(wrist_length, 2))}"
+            iyz="0.0"
+            izz="${(1.0/2.0) * wrist1_mass * pow(link_radius, 2)}"/>   <!-- inertia formula for cylinders (cylinder axis along z) -->
+        </inertial>
     </link>
     <joint name="wrist1" type="revolute">
@@ -128,4 +178,14 @@
             <material name="Black"/>
         </visual>
+        <inertial>
+            <mass value="${wrist2_joint_mass}"/>
+            <origin xyz="0.0 0.0 -${wrist2_radius/2}" rpy="0 0 0"/> <!-- position in the center -->
+            <inertia ixx="${(2.0/5.0) * wrist2_joint_mass * pow(wrist2_radius, 2)}"
+            ixy="0.0"
+            ixz="0.0"
+            iyy="${(2.0/5.0) * wrist2_joint_mass * pow(wrist2_radius, 2)}"
+            iyz="0.0"
+            izz="${(2.0/5.0) * wrist2_joint_mass * pow(wrist2_radius, 2)}"/>   <!-- inertia formula for spheres -->
+        </inertial>
     </link>
     <joint name="wrist2" type="revolute">
@@ -152,4 +212,15 @@
             <material name="Black"/>
         </visual>
+        <inertial>      <!-- to simplify we approximate the inertia computation to a cylinder with the mic sphere's radius -->
+            <mass value="${mic_mass}"/>
+            <origin xyz="0 0 -0.08" rpy="0 0 0"/> <!-- center in the center of the approx cylinder (sphere radius+cylinder length)/2 -->
+            <inertia
+                ixx="${(1.0/12.0) * mic_mass * (3*pow(0.03,2) + pow(0.08,2))}"
+                ixy="0.0"
+                ixz="0.0"
+                iyy="${(1.0/12.0) * mic_mass * (3*pow(0.03,2) + pow(0.08,2))}"
+                iyz="0.0"
+                izz="${(1.0/2.0) * mic_mass * pow(0.03,2)}"/>
+        </inertial>
     </link>
     <joint name="mic_frame" type="fixed">
